File: hardware/kicad/cupwarmer-hw/heater-control.kicad_sch (KiCad schematic)
At the start: 13 parts, among them Q1 AO3400 SOT-23

Commit message: Upgrade R3 shunt footprint from 0603 to 1206 for 0.05R bring-up
Phase 3-3 of docs/plans/20260509-pcb-dual-review-fixes.md.

R3 sits in the heater current path: 0R for production, 0.05R during
bring-up to read I_HEATER_MON on a scope. At 1.4 A peak, 0.05R
dissipates ~100 mW, which has zero margin in 0603 (1/10 W). 1206 gives
4x derating and accommodates a dedicated current-sense part with a
useful TC.

- heater-control.kicad_sch: R3 footprint -> R_1206_3216Metric;
  production LCSC C17888 (1206W4F0000T5E, 0R 1206 Basic);
  Description annotates bring-up MPN FRM121WFR050TM (LCSC C7467249,
  1W 1206 +/-1% +/-50ppm) sourced from JLCPCB.
- cupwarmer-hw.kicad_pcb: pcb sync swapped R3 to 1206 footprint;
  manual reroute of HEATER_OUT and Q1 reference field done in KiCad
  to clear the larger 1206 pads. DRC: 0 errors / 0 unconnected
  (1 lib_footprint_mismatch warning, benign local override).

Co-Authored-By: Claude Opus 4.7 (1M context) <noreply@anthropic.com>
Parts:
- R3: footprint Resistor_SMD:R_0603_1608Metric -> Resistor_SMD:R_1206_3216Metric; LCSC C21189 -> C17888; MPN 0603WAF0000T5E -> 1206W4F0000T5E
Changed lines of the file:
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@@
 			)
 		)
-		(property "Footprint" "Resistor_SMD:R_0603_1608Metric"
+		(property "Footprint" "Resistor_SMD:R_1206_3216Metric"
 			(at 115.57 119.38 90)
 			(hide yes)
@@
 			)
 		)
-		(property "Description" "Fit 0R for v1 normal build; substitute 0.05R for measured bring-up"
+		(property "Description" "Fit 0R for v1 normal build (C17888); substitute 0.05R 1W FRM121WFR050TM (C7467249) for measured bring-up"
 			(at 115.57 119.38 90)
 			(hide yes)
@@
 			)
 		)
-		(property "LCSC" "C21189"
+		(property "LCSC" "C17888"
 			(at 19.05 17.78 0)
 			(hide yes)
@@
 			)
 		)
-		(property "MPN" "0603WAF0000T5E"
+		(property "MPN" "1206W4F0000T5E"
 			(at 19.05 17.78 0)
 			(hide yes)
