File: hardware/kicad/cupwarmer-hw/heater-control.kicad_sch (KiCad schematic)
At the start: 13 parts, among them Q1 AO3400 SOT-23

Commit message: Reduce I2C testpads to single TP1
Remove the duplicate testpad and rename the remaining one to TP1.

Co-Authored-By: Claude Opus 4.7 (1M context) <noreply@anthropic.com>
Parts:
- removed TP1: TP_NTC, Connector_PinHeader_2.54mm:PinHeader_1x01_P2.54mm_Vertical, symbol cupwarmer:TESTPAD_1
- renumbered TP2 to TP1
Changed lines of the file:
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@@
-	)
-	(junction
-		(at 72.39 62.23)
-		(diameter 0)
-		(color 0 0 0 0)
 	)
 	(junction
@@
 		(pts
 			(xy 176.53 62.23) (xy 175.26 62.23)
-		)
-		(stroke
-			(width 0)
-			(type default)
-		)
-	)
-	(wire
-		(pts
-			(xy 72.39 62.23) (xy 72.39 63.5)
 		)
 		(stroke
@@
 		(in_pos_files no)
 		(dnp no)
-		(property "Reference" "TP2"
+		(property "Reference" "TP1"
 			(at 124.46 139.7 0)
 			(show_name no)
@@
 			(project "cupwarmer-hw"
 				(path "/f3c63676-f392-4700-9f58-a6787e1eb284/22222222-2222-2222-2222-222222222222"
-					(reference "TP2")
+					(reference "TP1")
 					(unit 1)
 				)
@@
 					(unit 1)
 				)
-			)
-		)
-	)
-	(symbol
-		(lib_id "cupwarmer:TESTPAD_1")
-		(at 72.39 68.58 0)
-		(unit 1)
-		(body_style 1)
-		(exclude_from_sim no)
-		(in_bom no)
-		(on_board yes)
-		(in_pos_files no)
-		(dnp no)
-		(property "Reference" "TP1"
-			(at 72.39 71.12 0)
-			(show_name no)
-			(do_not_autoplace no)
-			(effects
-				(font
-					(size 1.27 1.27)
-				)
-			)
-		)
-		(property "Value" "TP_NTC"
-			(at 67.58 68.25 0)
-			(show_name no)
-			(do_not_autoplace no)
-			(effects
-				(font
-					(size 1.27 1.27)
-				)
-			)
-		)
-		(property "Footprint" "Connector_PinHeader_2.54mm:PinHeader_1x01_P2.54mm_Vertical"
-			(at 72.39 68.58 0)
-			(hide yes)
-			(show_name no)
-			(do_not_autoplace no)
-			(effects
-				(font
-					(size 1.27 1.27)
-				)
-			)
-		)
-		(property "Datasheet" "~"
-			(at 72.39 68.58 0)
-			(hide yes)
-			(show_name no)
-			(do_not_autoplace no)
-			(effects
-				(font
-					(size 1.27 1.27)
-				)
-			)
-		)
-		(property "Description" "DMM probe pad for heater NTC before powered test"
-			(at 72.39 68.58 0)
-			(hide yes)
-			(show_name no)
-			(do_not_autoplace no)
-			(effects
-				(font
-					(size 1.27 1.27)
-				)
-			)
-		)
-		(pin "1"
-		)
-		(instances
-			(project "cupwarmer-hw"
-				(path "/f3c63676-f392-4700-9f58-a6787e1eb284/22222222-2222-2222-2222-222222222222"
-					(reference "TP1")
-					(unit 1)
-				)

Commit message: Add M2 plastic-screw bosses on PCB support ribs
Add a cylindrical M2 self-tap boss (φ5, pilot φ1.7, 4mm deep) on top of
each of the 4 PCB support ribs in the enclosure, hulled with the rib for
a smooth tangent blend and inset 0.5mm outward from the rib inner face
so the boss does not protrude into the L1 coil envelope.

Add 2 NPTH φ2.4 mounting holes (H1, H2) on the PCB that match the boss
positions. Rename the existing heater-harness footprint H1→J2 to free
up the H prefix for the new mounting holes, and rename the off-board
heater-side connector H2→J3 in the schematic for consistency.

Co-Authored-By: Claude Opus 4.7 (1M context) <noreply@anthropic.com>
Parts:
- renumbered H1 to J2, H2 to J3
Changed lines of the file:
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@@
 		(in_pos_files yes)
 		(dnp no)
-		(property "Reference" "H1"
+		(property "Reference" "J2"
 			(at 146.558 54.61 0)
 			(show_name no)
@@
 			(project "cupwarmer-hw"
 				(path "/f3c63676-f392-4700-9f58-a6787e1eb284/22222222-2222-2222-2222-222222222222"
-					(reference "H1")
+					(reference "J2")
 					(unit 1)
 				)
@@
 		(in_pos_files yes)
 		(dnp no)
-		(property "Reference" "H2"
+		(property "Reference" "J3"
 			(at 165.862 54.61 0)
 			(show_name no)
@@
 			(project "cupwarmer-hw"
 				(path "/f3c63676-f392-4700-9f58-a6787e1eb284/22222222-2222-2222-2222-222222222222"
-					(reference "H2")
+					(reference "J3")
 					(unit 1)
 				)
