File: hardware/kicad/cupwarmer-hw/heater-control.kicad_sch (KiCad schematic)
At the start: 12 parts, among them J2 4-pin heater lead pcb side, J3 4-pin heater lead heater side, Q1 AO3400 SOT-23

Commit message: Update PCBA BOM and fabrication outputs
Parts:
- F1: value KSD9700-70/5JSB/080C -> NR72CB0; LCSC C156512 -> C183007; MPN KSD9700-70/5JSB/080C -> NR72CB0; Manufacturer Xucheng Elec -> Bourns
Changed lines of the file:
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@@
 			)
 		)
-		(property "Value" "KSD9700-70/5JSB/080C"
+		(property "Value" "NR72CB0"
 			(at 193.04 34.036 0)
 			(show_name no)
@@
 			)
 		)
-		(property "Description" "Independent thermal cutoff in series before heater"
+		(property "Description" "Independent low-profile 12V heater thermal cutoff"
 			(at 193.04 40.64 0)
 			(hide yes)
@@
 			)
 		)
-		(property "Manufacturer" "Xucheng Elec"
+		(property "Manufacturer" "Bourns"
 			(at 137.16 -17.78 0)
 			(hide yes)
@@
 			)
 		)
-		(property "LCSC" "C156512"
+		(property "LCSC" "C183007"
 			(at 137.16 -17.78 0)
 			(hide yes)
@@
 			)
 		)
-		(property "MPN" "KSD9700-70/5JSB/080C"
+		(property "MPN" "NR72CB0"
 			(at 137.16 -17.78 0)
 			(hide yes)
