File: hardware/kicad/cupwarmer-hw/heater-control.kicad_sch (KiCad schematic)
At the start: 12 parts, among them J2 4-pin heater lead pcb side, J3 4-pin heater lead heater side, Q1 AO3400 SOT-23

Commit message: Align C18/C19 & R3 parts, reconcile BOM/CPL with PCB, regen fab
- C18/C19: YAGEO NP0 CC0603JRNPO9BN103 (C389113) -> Murata C0G
  GRM1885C1H103JA01D (C85973), unifying with C11/C13 (sch/pcb/bom)
- R3: default to 0.05R 1W FRM121WFR050TM (C7467249) bring-up shunt;
  0R 1206 jumper kept as production alternate (sch/pcb)
- Z1/Z3/Z4 TVS rotation/polarity reflected in PCB + CPL; gerbers regenerated
- BOM: rename heater-harness ref H1 -> J2 to match PCB; merge C11/C13 into
  one row; note J1 as hand-soldered THT excluded from CPL
- CPL: drop non-assembled parts (J1, J2, L1) and fiducials (FID1-3);
  45 SMT placements remain
- Verified BOM <-> jlcpcb-bom <-> CPL <-> PCB parity: designators, LCSC,
  and values all consistent

Co-Authored-By: Claude Opus 4.8 (1M context) <noreply@anthropic.com>
Parts:
- R3: LCSC C17888 -> C7467249; MPN 1206W4F0000T5E -> FRM121WFR050TM; Manufacturer UNI-ROYAL -> FOJAN
Changed lines of the file:
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@@
 			)
 		)
-		(property "Description" "Fit 0R for v1 normal build (C17888); substitute 0.05R 1W FRM121WFR050TM (C7467249) for measured bring-up"
+		(property "Description" "Fit 0.05R 1W FRM121WFR050TM (C7467249) for measured bring-up; production build may substitute 0R 1206 jumper C17888 / 1206W4F0000T5E"
 			(at 115.57 119.38 90)
 			(hide yes)
@@
 			)
 		)
-		(property "Manufacturer" "UNI-ROYAL"
+		(property "Manufacturer" "FOJAN"
 			(at 19.05 17.78 0)
 			(hide yes)
@@
 			)
 		)
-		(property "LCSC" "C17888"
+		(property "LCSC" "C7467249"
 			(at 19.05 17.78 0)
 			(hide yes)
@@
 			)
 		)
-		(property "MPN" "1206W4F0000T5E"
+		(property "MPN" "FRM121WFR050TM"
 			(at 19.05 17.78 0)
 			(hide yes)
