File: hardware/kicad/cupwarmer-hw/sensors-logic.kicad_sch (KiCad schematic)
At the start: 6 parts, among them J1 I2C Service, J2 THERM_MON, J3 STATUS_MON

Commit message: Align cupwarmer BOM with STEVAL-WLC38RX reference (JLCPCB-orderable)
- Pick concrete JLCPCB MPNs for all TBD parts in initial-bom.csv:
  - Cs (5x 100nF) and 100nF bypass roles → Wuerth 885012206095 (C6715111),
    matching STEVAL exactly.
  - 10uF rectifier/output bulk → Murata GRM188R6YA106MA73D (C194427).
  - 4.7uF VAA → Murata GRM188R61E475KE11D (C90057).
  - Add VRECT/VOUT bulk + HF + Z4 SMBJ18A clamp per STEVAL UM3154.
  - Other passives: Samsung MLCC, UNI-ROYAL 0603 1% resistors,
    KEXIN 10k NTC, SMF13A/SMBJ15A TVS, AO3400, KSD9700-70.
- Add `lcsc` column to BOM CSV; mark mechanical/board-feature rows.
- Sync MPN/LCSC/Manufacturer properties onto every schematic symbol via
  tmp/apply_bom_properties.py (idempotent helper).
- pcb_netlist.py: always seed fp-lib-table from stock template so system
  libraries resolve when the global table is just a Table-type indirection.
- design-notes: document VRECT/VOUT cap network and Z3/Z4 TVS choices.
- CLAUDE.md / wiki/README.md: point at ./wiki/ as the project's reference
  store.

Co-Authored-By: Claude Opus 4.7 (1M context) <noreply@anthropic.com>
Parts:
- J1: LCSC (none) -> C2691448; MPN (none) -> PZ254V-11-04P; Manufacturer (none) -> Boom Precision
- J2, J3: LCSC (none) -> C492401; MPN (none) -> PZ254V-11-02P; Manufacturer (none) -> Boom Precision
- R8: LCSC (none) -> C25804; MPN (none) -> 0603WAF1002T5E; Manufacturer (none) -> UNI-ROYAL
- TH1, TH2: LCSC (none) -> C2892547; MPN (none) -> KNTC0603/10KF3950; Manufacturer (none) -> KEXIN
Changed lines of the file:
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@@
+			)
+		)
+		(property "Manufacturer" "Boom Precision"
+			(at 0 0 0)
+			(hide yes)
+			(show_name no)
+			(do_not_autoplace no)
+			(effects
+				(font
+					(size 1.27 1.27)
+				)
+			)
+		)
+		(property "LCSC" "C492401"
+			(at 0 0 0)
+			(hide yes)
+			(show_name no)
+			(do_not_autoplace no)
+			(effects
+				(font
+					(size 1.27 1.27)
+				)
+			)
+		)
+		(property "MPN" "PZ254V-11-02P"
+			(at 0 0 0)
+			(hide yes)
+			(show_name no)
+			(do_not_autoplace no)
+			(effects
+				(font
+					(size 1.27 1.27)
+				)
 			)
 		)
@@
 			)
 		)
+		(property "Manufacturer" "Boom Precision"
+			(at 0 0 0)
+			(hide yes)
+			(show_name no)
+			(do_not_autoplace no)
+			(effects
+				(font
+					(size 1.27 1.27)
+				)
+			)
+		)
+		(property "LCSC" "C2691448"
+			(at 0 0 0)
+			(hide yes)
+			(show_name no)
+			(do_not_autoplace no)
+			(effects
+				(font
+					(size 1.27 1.27)
+				)
+			)
+		)
+		(property "MPN" "PZ254V-11-04P"
+			(at 0 0 0)
+			(hide yes)
+			(show_name no)
+			(do_not_autoplace no)
+			(effects
+				(font
+					(size 1.27 1.27)
+				)
+			)
+		)
 		(pin "1"
 		)
@@
 			)
 		)
+		(property "Manufacturer" "KEXIN"
+			(at 0 0 0)
+			(hide yes)
+			(show_name no)
+			(do_not_autoplace no)
+			(effects
+				(font
+					(size 1.27 1.27)
+				)
+			)
+		)
+		(property "LCSC" "C2892547"
+			(at 0 0 0)
+			(hide yes)
+			(show_name no)
+			(do_not_autoplace no)
+			(effects
+				(font
+					(size 1.27 1.27)
+				)
+			)
+		)
+		(property "MPN" "KNTC0603/10KF3950"
+			(at 0 0 0)
+			(hide yes)
+			(show_name no)
+			(do_not_autoplace no)
+			(effects
+				(font
+					(size 1.27 1.27)
+				)
+			)
+		)
 		(pin "1"
 		)
@@
 			)
 		)
+		(property "Manufacturer" "KEXIN"
+			(at 0 0 0)
+			(hide yes)
+			(show_name no)
+			(do_not_autoplace no)
+			(effects
+				(font
+					(size 1.27 1.27)
+				)
+			)
+		)
+		(property "LCSC" "C2892547"
+			(at 0 0 0)
+			(hide yes)
+			(show_name no)
+			(do_not_autoplace no)
+			(effects
+				(font
+					(size 1.27 1.27)
+				)
+			)
+		)
+		(property "MPN" "KNTC0603/10KF3950"
+			(at 0 0 0)
+			(hide yes)
+			(show_name no)
+			(do_not_autoplace no)
+			(effects
+				(font
+					(size 1.27 1.27)
+				)
+			)
+		)
 		(pin "1"
 		)
@@
 			)
 		)
+		(property "Manufacturer" "Boom Precision"
+			(at 0 0 0)
+			(hide yes)
+			(show_name no)
+			(do_not_autoplace no)
+			(effects
+				(font
+					(size 1.27 1.27)
+				)
+			)
+		)
+		(property "LCSC" "C492401"
+			(at 0 0 0)
+			(hide yes)
+			(show_name no)
+			(do_not_autoplace no)
+			(effects
+				(font
+					(size 1.27 1.27)
+				)
+			)
+		)
+		(property "MPN" "PZ254V-11-02P"
+			(at 0 0 0)
+			(hide yes)
+			(show_name no)
+			(do_not_autoplace no)
+			(effects
+				(font
+					(size 1.27 1.27)
+				)
+			)
+		)
 		(pin "1"
 		)
@@
 			(hide yes)
 			(show_name no)
+			(do_not_autoplace no)
+			(effects
+				(font
+					(size 1.27 1.27)
+				)
+			)
+		)
+		(property "Manufacturer" "UNI-ROYAL"
+			(at 0 0 0)
+			(hide yes)
+			(show_name no)
+			(do_not_autoplace no)
+			(effects
+				(font
+					(size 1.27 1.27)
+				)
+			)
+		)
+		(property "LCSC" "C25804"
+			(at 0 0 0)
+			(hide yes)
+			(show_name no)
+			(do_not_autoplace no)
+			(effects
+				(font
+					(size 1.27 1.27)
+				)
+			)
+		)
+		(property "MPN" "0603WAF1002T5E"
+			(at 0 0 0)
+			(hide yes)
+			(show_name no)

Commit message: Apply ST UM3154 review fixes to Qi RX schematic
Address tape-out blockers from STEVAL-WLC38RX (UM3154) reference diff:

- Add R12 (10k) INTB pullup to RX_VAA on rx-power
- Add R13 (10k) ENB pulldown to SYS_GND on rx-power
  (replaces direct ENB->GND tie; matches ST eval, allows future MCU control)
- C18, C19 value 100nF -> 10nF (NP0) on rx-power
  (Cs=320nF total with 8uH coil targets ~99.5kHz Qi resonance vs prior 79.6kHz)
- Replace TH2 with Murata NCP18WF104F12RB 100k B25/85=4260K on sensors-logic
  (matches ST eval reference 100k NTC; aligns with default HOTP threshold)
- Remove TH1 + R8 + J2 (THERM_MON) and NTC_TOP labels from sensors-logic
  (redundant; KSD9700 + STWLC38 HOTP via TH2 already provide thermal protection)
- BOM: add R12, R13; replace TH2 entry; split C1/16/17/18/19 into two rows;
  drop TH1, R8, J2; tweak R7 description
- heater-control: H1 Value text updated to "12R 12W Heater (external)"

ERC: 0 errors, 0 warnings.

Co-Authored-By: Claude Opus 4.7 (1M context) <noreply@anthropic.com>
Parts:
- removed J2: THERM_MON, Connector_PinHeader_2.54mm:PinHeader_1x02_P2.54mm_Vertical, symbol cupwarmer:PASSIVE_2
- removed R8: 10k Pull-up, Resistor_SMD:R_0603_1608Metric, symbol cupwarmer:PASSIVE_2
- removed TH1: NTC 10k B3950, Connector_Wire:SolderWire-0.1sqmm_1x02_P3.6mm_D0.4mm_OD1mm_Relief2x, symbol cupwarmer:PASSIVE_2
- TH2: value NTC 10k B3950 -> NTC 100k B4250; LCSC C2892547 -> C71280; MPN KNTC0603/10KF3950 -> NCP18WF104F12RB; Manufacturer KEXIN -> Murata Electronics
