File: hardware/kicad/cupwarmer-hw/rx-power.kicad_sch (KiCad schematic)
At the start: 40 parts, among them J1 I2C Service, J3 STATUS_MON, U1 STWLC38JRM

Commit message: Swap Cs primary caps to C0G 1206 (3x100nF GRM31C5C1H104JA01L)
C1/C16/C17 were 100nF/50V X7R 0603 (Würth 885012206095). cup warmer is
in continuous warm operation (heater H1 + coil losses), so the X7R
temperature drift (+/-15%) plus DC bias capacitance loss would shift
the AC series resonance and degrade efficiency / VRECT regulation.
C0G (NP0, +/-30 ppm/degC, no DC-bias drop) is required.

JLC DB confirmed 100nF/50V C0G is unavailable in 0603 and 0805
(C0G volumetric efficiency caps 0805 50V at ~33nF). 1206 is the
smallest stocked size for 100nF/50V C0G; 3x1206 (15.4 mm^2) beats
14x22nF/0805 (35 mm^2) on total board area, so going up in package
size for fewer parts is the right trade-off here.

Footprint pitch widened from 1.5 mm to 2.5 mm to clear 1206 courtyards
(C1@85.5/82, C16@88/82, C17@90.5/82, all rotation 90, C18/C19 retained
at 92.5/94). DRC violation count drops from 231 to 212 with the three
courtyards_overlap entries for C1/C16/C17 cleared. Net topology
preserved (verified via netlist diff: Net-(C1-Pad1)=L1.2+caps,
Net-(C1-Pad2)=U1.AC1+caps unchanged). C18/C19 (10nF NP0 0603) and
unrelated 885012206095 instances (C4/C22/C24 bypass caps) untouched.

Co-Authored-By: Claude Opus 4.7 (1M context) <noreply@anthropic.com>
Parts:
- C1, C16, C17: footprint Capacitor_SMD:C_0603_1608Metric -> Capacitor_SMD:C_1206_3216Metric; LCSC C6715111 -> C97946; MPN 885012206095 -> GRM31C5C1H104JA01L; Manufacturer Wuerth Elektronik -> Murata
Changed lines of the file:
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@@
 			)
 		)
-		(property "Footprint" "Capacitor_SMD:C_0603_1608Metric"
+		(property "Footprint" "Capacitor_SMD:C_1206_3216Metric"
 			(at 64.77 76.2 0)
 			(hide yes)
@@
 			)
 		)
-		(property "Description" "Resonant capacitor, one of five parallel 100nF C0G parts"
+		(property "Description" "100nF 50V C0G +/-5%"
 			(at 64.77 76.2 0)
 			(hide yes)
@@
 			)
 		)
-		(property "Manufacturer" "Wuerth Elektronik"
-			(at 0 0 0)
-			(hide yes)
-			(show_name no)
-			(do_not_autoplace no)
-			(effects
-				(font
-					(size 1.27 1.27)
-				)
-			)
-		)
-		(property "LCSC" "C6715111"
-			(at 0 0 0)
-			(hide yes)
-			(show_name no)
-			(do_not_autoplace no)
-			(effects
-				(font
-					(size 1.27 1.27)
-				)
-			)
-		)
-		(property "MPN" "885012206095"
+		(property "Manufacturer" "Murata"
+			(at 0 0 0)
+			(hide yes)
+			(show_name no)
+			(do_not_autoplace no)
+			(effects
+				(font
+					(size 1.27 1.27)
+				)
+			)
+		)
+		(property "LCSC" "C97946"
+			(at 0 0 0)
+			(hide yes)
+			(show_name no)
+			(do_not_autoplace no)
+			(effects
+				(font
+					(size 1.27 1.27)
+				)
+			)
+		)
+		(property "MPN" "GRM31C5C1H104JA01L"
 			(at 0 0 0)
 			(hide yes)
@@
 			)
 		)
-		(property "Footprint" "Capacitor_SMD:C_0603_1608Metric"
+		(property "Footprint" "Capacitor_SMD:C_1206_3216Metric"
 			(at 64.77 81.28 0)
 			(hide yes)
@@
 			)
 		)
-		(property "Description" "Resonant capacitor, one of five parallel 100nF C0G parts"
+		(property "Description" "100nF 50V C0G +/-5%"
 			(at 64.77 81.28 0)
 			(hide yes)
@@
 			)
 		)
-		(property "Manufacturer" "Wuerth Elektronik"
-			(at 0 0 0)
-			(hide yes)
-			(show_name no)
-			(do_not_autoplace no)
-			(effects
-				(font
-					(size 1.27 1.27)
-				)
-			)
-		)
-		(property "LCSC" "C6715111"
-			(at 0 0 0)
-			(hide yes)
-			(show_name no)
-			(do_not_autoplace no)
-			(effects
-				(font
-					(size 1.27 1.27)
-				)
-			)
-		)
-		(property "MPN" "885012206095"
+		(property "Manufacturer" "Murata"
+			(at 0 0 0)
+			(hide yes)
+			(show_name no)
+			(do_not_autoplace no)
+			(effects
+				(font
+					(size 1.27 1.27)
+				)
+			)
+		)
+		(property "LCSC" "C97946"
+			(at 0 0 0)
+			(hide yes)
+			(show_name no)
+			(do_not_autoplace no)
+			(effects
+				(font
+					(size 1.27 1.27)
+				)
+			)
+		)
+		(property "MPN" "GRM31C5C1H104JA01L"
 			(at 0 0 0)
 			(hide yes)
@@
 			)
 		)
-		(property "Footprint" "Capacitor_SMD:C_0603_1608Metric"
+		(property "Footprint" "Capacitor_SMD:C_1206_3216Metric"
 			(at 64.77 86.36 0)
 			(hide yes)
@@
 			)
 		)
-		(property "Description" "Resonant capacitor, one of five parallel 100nF C0G parts"
+		(property "Description" "100nF 50V C0G +/-5%"
 			(at 64.77 86.36 0)
 			(hide yes)
@@
 			)
 		)
-		(property "Manufacturer" "Wuerth Elektronik"
-			(at 0 0 0)
-			(hide yes)
-			(show_name no)
-			(do_not_autoplace no)
-			(effects
-				(font
-					(size 1.27 1.27)
-				)
-			)
-		)
-		(property "LCSC" "C6715111"
-			(at 0 0 0)
-			(hide yes)
-			(show_name no)
-			(do_not_autoplace no)
-			(effects
-				(font
-					(size 1.27 1.27)
-				)
-			)
-		)
-		(property "MPN" "885012206095"
-			(at 0 0 0)
-			(hide yes)
+		(property "Manufacturer" "Murata"
+			(at 0 0 0)
+			(hide yes)
+			(show_name no)
+			(do_not_autoplace no)
+			(effects
+				(font
+					(size 1.27 1.27)
+				)
+			)
+		)
+		(property "LCSC" "C97946"
+			(at 0 0 0)
+			(hide yes)
+			(show_name no)
+			(do_not_autoplace no)
+			(effects
+				(font
+					(size 1.27 1.27)
+				)
+			)
+		)
+		(property "MPN" "GRM31C5C1H104JA01L"
+			(at 0 0 0)
+			(hide yes)
