File: hardware/kicad/cupwarmer-hw/rx-power.kicad_sch (KiCad schematic)
At the start: 41 parts, among them J1 I2C Service, J3 STATUS_MON, U1 STWLC38JRM

Commit message: Pour SYS_GND on inner layers and label rx-power nets
- PCB: add SYS_GND zones on In1.Cu/In2.Cu, add GND stitching vias,
  reflow footprint placement
- rx-power.sch: label AC1/2, COMA1/2, COMB1/2, BOOT1/2, VRECT nets
- heater-control.sch: nudge KSD9700 value label
- project: housekeeping from KiCad open

Co-Authored-By: Claude Opus 4.7 (1M context) <noreply@anthropic.com>
Connections:
- net AC2: now reaches C13.1, C14.1, C6.1, L1.1, U1.B1 (AC2), U1.B2 (AC2), U1.C1 (AC2), U1.C2 (AC2), Z2.1
- net COMB2: now reaches C14.2, U1.H2 (COMB2)
- net VRECT: now reaches C20.1, C21.1, C22.1, C9.1, R14.2, R4.2, U1.D1 (VRECT), U1.D2 (VRECT), U1.D3 (VRECT), U1.D4 (VRECT), U1.D5 (VRECT), Z4.2
- net AC1: now reaches C1.2, C11.1, C12.1, C16.2, C17.2, C18.2, C19.2, C5.1, U1.B4 (AC1), U1.B5 (AC1), U1.C4 (AC1), U1.C5 (AC1), Z1.2
- net BOOT1: now reaches C5.2, U1.B3 (BOOT1)
- net BOOT2: now reaches C6.2, U1.C3 (BOOT2)
- net COMA1: now reaches C11.2, U1.G1 (COMA1)
- net COMA2: now reaches C13.2, U1.G2 (COMA2)
- net COMB1: now reaches C12.2, U1.H1 (COMB1)
Changed lines of the file:
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@@
+	)
+	(junction
+		(at 232.41 87.63)
+		(diameter 0)
+		(color 0 0 0 0)
 	)
 	(junction
@@
 	(wire
 		(pts
+			(xy 232.41 83.82) (xy 232.41 87.63)
+		)
+		(stroke
+			(width 0)
+			(type default)
+		)
+	)
+	(wire
+		(pts
 			(xy 114.3 128.27) (xy 109.22 128.27)
 		)
@@
 	(wire
 		(pts
-			(xy 204.47 87.63) (xy 236.22 87.63)
+			(xy 204.47 87.63) (xy 232.41 87.63)
 		)
 		(stroke
@@
 	(wire
 		(pts
+			(xy 232.41 87.63) (xy 236.22 87.63)
+		)
+		(stroke
+			(width 0)
+			(type default)
+		)
+	)
+	(wire
+		(pts
 			(xy 109.22 128.27) (xy 109.22 125.73)
 		)
@@
 		)
 	)
+	(label "COMB2"
+		(at 116.84 118.11 0)
+		(effects
+			(font
+				(size 1.27 1.27)
+			)
+			(justify left bottom)
+		)
+	)
+	(label "AC2"
+		(at 88.9 113.03 0)
+		(effects
+			(font
+				(size 1.27 1.27)
+			)
+			(justify left bottom)
+		)
+	)
+	(label "BOOT1"
+		(at 118.11 87.63 0)
+		(effects
+			(font
+				(size 1.27 1.27)
+			)
+			(justify left bottom)
+		)
+	)
+	(label "BOOT2"
+		(at 119.38 120.65 0)
+		(effects
+			(font
+				(size 1.27 1.27)
+			)
+			(justify left bottom)
+		)
+	)
+	(label "COMA2"
+		(at 114.3 115.57 0)
+		(effects
+			(font
+				(size 1.27 1.27)
+			)
+			(justify left bottom)
+		)
+	)
+	(label "COMA1"
+		(at 113.03 92.71 0)
+		(effects
+			(font
+				(size 1.27 1.27)
+			)
+			(justify left bottom)
+		)
+	)
+	(label "COMB1"
+		(at 115.57 90.17 0)
+		(effects
+			(font
+				(size 1.27 1.27)
+			)
+			(justify left bottom)
+		)
+	)
+	(label "VRECT"
+		(at 232.41 83.82 0)
+		(effects
+			(font
+				(size 1.27 1.27)
+			)
+			(justify left bottom)
+		)
+	)
+	(label "AC1"
+		(at 88.9 95.25 0)
+		(effects
+			(font
+				(size 1.27 1.27)
+			)
+			(justify left bottom)
+		)
+	)
