File: hardware/kicad/cupwarmer-hw/rx-power.kicad_sch (KiCad schematic)
At the start: 40 parts, among them J1 I2C Service, J3 STATUS_MON, U1 STWLC38JRM

Commit message: Remove R7 from rx-power after move to heater-control
R7 was relocated to the heater-control sheet in 7f9c5df; clean up
the rx-power side by deleting the symbol, the now-unused junction
and wire stub, and re-anchoring the RX_VAA / RX_NTC global labels.

Co-Authored-By: Claude Opus 4.7 (1M context) <noreply@anthropic.com>
Parts:
- removed R7: 51k, Resistor_SMD:R_0603_1608Metric, symbol cupwarmer:PASSIVE_2
Changed lines of the file:
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@@
 	)
 	(junction
-		(at 144.78 132.08)
-		(diameter 0)
-		(color 0 0 0 0)
-	)
-	(junction
 		(at 102.87 113.03)
 		(diameter 0)
@@
 	(wire
 		(pts
-			(xy 134.62 132.08) (xy 144.78 132.08)
+			(xy 142.24 132.08) (xy 144.78 132.08)
 		)
 		(stroke
@@
 	(wire
 		(pts
-			(xy 144.78 142.24) (xy 157.48 142.24)
-		)
-		(stroke
-			(width 0)
-			(type default)
-		)
-	)
-	(wire
-		(pts
 			(xy 96.52 113.03) (xy 96.52 115.57)
 		)
@@
 	(global_label "RX_VAA"
 		(shape passive)
-		(at 144.78 142.24 270)
+		(at 157.48 142.24 0)
 		(effects
 			(font
 				(size 1.27 1.27)
 			)
-			(justify right)
+			(justify left)
 		)
 		(property "Intersheetrefs" "${INTERSHEET_REFS}"
-			(at 144.78 142.24 90)
+			(at 157.48 142.24 0)
 			(hide yes)
 			(show_name no)
@@
 	(global_label "RX_NTC"
 		(shape bidirectional)
-		(at 134.62 132.08 180)
+		(at 142.24 132.08 180)
 		(effects
 			(font
@@
 		)
 		(property "Intersheetrefs" "${INTERSHEET_REFS}"
-			(at 134.62 132.08 0)
+			(at 142.24 132.08 0)
 			(hide yes)
 			(show_name no)
@@
 					(unit 1)
 				)
-			)
-		)
-	)
-	(symbol
-		(lib_id "cupwarmer:PASSIVE_2")
-		(at 144.78 137.16 270)
-		(unit 1)
-		(body_style 1)
-		(exclude_from_sim no)
-		(in_bom yes)
-		(on_board yes)
-		(in_pos_files yes)
-		(dnp no)
-		(property "Reference" "R7"
-			(at 148.59 137.16 0)
-			(show_name no)
-			(do_not_autoplace no)
-			(effects
-				(font
-					(size 1.27 1.27)
-				)
-			)
-		)
-		(property "Value" "51k"
-			(at 141.224 137.16 180)
-			(show_name no)
-			(do_not_autoplace no)
-			(effects
-				(font
-					(size 1.27 1.27)
-				)
-			)
-		)
-		(property "Footprint" "Resistor_SMD:R_0603_1608Metric"
-			(at 144.78 137.16 180)
-			(hide yes)
-			(show_name no)
-			(do_not_autoplace no)
-			(effects
-				(font
-					(size 1.27 1.27)
-				)
-			)
-		)
-		(property "Datasheet" "~"
-			(at 144.78 137.16 180)
-			(hide yes)
-			(show_name no)
-			(do_not_autoplace no)
-			(effects
-				(font
-					(size 1.27 1.27)
-				)
-			)
-		)
-		(property "Description" "NTC pull-up to RX_VAA (51k); forms divider with external 100k/B4260 heater NTC on RX_NTC for STWLC38 OTP (~69C typ, VNTC,OTP=0.59V)"
-			(at 144.78 137.16 180)
-			(hide yes)
-			(show_name no)
-			(do_not_autoplace no)
-			(effects
-				(font
-					(size 1.27 1.27)
-				)
-			)
-		)
-		(property "Manufacturer" "UNI-ROYAL"
-			(at 0 0 0)
-			(hide yes)
-			(show_name no)
-			(do_not_autoplace no)
-			(effects
-				(font
-					(size 1.27 1.27)
-				)
-			)
-		)
-		(property "LCSC" "C23196"
-			(at 0 0 0)
-			(hide yes)
-			(show_name no)
-			(do_not_autoplace no)
-			(effects
-				(font
-					(size 1.27 1.27)
-				)
-			)
-		)
-		(property "MPN" "0603WAF5102T5E"
-			(at 0 0 0)
-			(hide yes)
-			(show_name no)
-			(do_not_autoplace no)
-			(effects
-				(font
-					(size 1.27 1.27)
-				)
-			)
-		)
-		(pin "1"
-		)
-		(pin "2"
-		)
-		(instances
-			(project "rx-power"
-				(path "/11111111-aaaa-bbbb-cccc-111111111111"
-					(reference "R7")
-					(unit 1)
-				)
-			)
-			(project "cupwarmer-hw"
-				(path "/f3c63676-f392-4700-9f58-a6787e1eb284/11111111-1111-1111-1111-111111111111"
-					(reference "R7")
-					(unit 1)
-				)

Commit message: Replace J3 bring-up header with TP3 test pad on I_HEATER_MON
Drop the dual-purpose 2-pin J3 (RX_INTB + I_HEATER_MON bring-up) and
expose only I_HEATER_MON via a single-pin TP3 test pad matching
TP1/TP2 (TESTPAD_1 symbol, 1x01 pin header footprint). RX_INTB stays
internal to the U1.H4 ↔ R12.1 path with its label moved onto that
net.

Co-Authored-By: Claude Opus 4.7 (1M context) <noreply@anthropic.com>
Parts:
- removed J3: STATUS_MON, Connector_PinHeader_2.54mm:PinHeader_1x02_P2.54mm_Vertical, symbol cupwarmer:PASSIVE_2
Connections:
- net RX_INTB: no longer names the net of R12.1, U1.H4 (INTB)
Other:
- moved on the sheet: R12, R13
