File: hardware/kicad/cupwarmer-hw/cupwarmer-hw.kicad_pcb (KiCad board)
At the start: 4 copper layers, 56 x 56 mm, 50 parts, among them J1 I2C Service, J3 STATUS_MON, Q1 AO3400 SOT-23, U1 STWLC38JRM

Commit message: Add heater harness NTC routing
Parts:
- removed TH2: NTC 100k B4250, Resistor_SMD:R_0603_1608Metric
- added TP1: TP_NTC, cupwarmer:TestPoint_Pad_D1.0mm_NoSilk, F.Cu at (94.2, 125.5)
- added TP2: TP_NTC_GND, cupwarmer:TestPoint_Pad_D1.0mm_NoSilk, F.Cu at (105.0, 125.5)
- H1: value 12R 12W Heater (external) -> 12R 12W Heater + 100k NTC; footprint Connector_Wire:SolderWire-1sqmm_1x02_P5.4mm_D1.4mm_OD2.7mm -> cupwarmer:SolderWire-HeaterHarness_1x04_P5.0mm_D1.4mm
Connections:
- R7 pad 1: Net-(U1-NTC) -> RX_NTC
- U1 pad F1: Net-(U1-NTC) -> RX_NTC
Routing:
- net RX_NTC: track 0.00 -> 54.8 mm, vias 0 -> 1
- net Net-(U1-NTC): track 10.7 -> 0.00 mm
- net SYS_GND: track 32.8 -> 34.3 mm, vias 27 -> 26
